Commit message: include camera color frame diretly in urdf

File: urdf/stretch.urdf (robot description, URDF)
Before this commit: robot stretch, 47 links, 46 joints
Links:
- added link camera_color_optical_frame
Joints:
- added joint camera_color_optical_joint: type fixed, parent link_head_tilt, child camera_color_optical_frame, origin xyz=0.031591 -0.0119208 0.0807607 rpy=-1.5737774 0.0071859 -1.6093517
